File: Hardware/RGB_ledstrip_controller.sch (KiCad schematic (older format))
At the start: 15 parts, among them J1 Conn_RGBWW, Q1 IRLZ44N, Q2 IRLZ44N, Q3 IRLZ44N, Q4 IRLZ44N, U1 WeMos_mini, U2 L7805

Commit message: Created screenshot for readme
Parts:
- U1: symbol custom:WeMos_mini -> RGB_ledstrip_controller-rescue:WeMos_mini-custom
Changed lines of the file:
@@
 EESchema Schematic File Version 4
 LIBS:RGB_ledstrip_controller-cache
-EELAYER 26 0
+EELAYER 29 0
 EELAYER END
 $Descr A4 11693 8268
@@
 $EndDescr
 $Comp
-L custom:WeMos_mini U1
+L RGB_ledstrip_controller-rescue:WeMos_mini-custom U1
 U 1 1 5B8C508B
 P 5950 3350
